File: RMTS.kicad_sch (KiCad schematic)
At the start: 83 parts, among them J1 Screw_Terminal_01x02, J10 CONN_02, J11 CONN_02, J12 CONN_02, J2 Programmer, J3 Screw_Terminal_01x03, J4 Screw_Terminal_01x04, J5 Screw_Terminal_01x02, J6 Screw_Terminal_01x02, J7 Micro_SD_Card_Det_Hirose_DM3AT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

Commit message: Have JLC populate more components
Parts:
- C2: LCSC C176662 -> C340737
- D3: LCSC (none) -> C552950; now in the parts list
- U2: LCSC (none) -> C511780; now in the parts list
- U3: LCSC (none) -> C2869313; now in the parts list
- U4: LCSC (none) -> C636381; now in the parts list
- U5, U6: LCSC C22113 -> C189217
- U8: LCSC C2841056 -> C2871822
Changed lines of the file:
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@@
 		(unit 1)
 		(exclude_from_sim no)
-		(in_bom no)
+		(in_bom yes)
 		(on_board yes)
 		(dnp no)
@@
 			)
 		)
+		(property "LCSC" "C511780"
+			(at 191.77 121.92 0)
+			(effects
+				(font
+					(size 1.27 1.27)
+				)
+				(hide yes)
+			)
+		)
 		(pin "1"
 		)
@@
 			)
 		)
-		(property "LCSC" "C176662"
+		(property "LCSC" "C340737"
 			(at 171.45 45.72 0)
 			(effects
@@
 		(unit 1)
 		(exclude_from_sim no)
-		(in_bom no)
+		(in_bom yes)
 		(on_board yes)
 		(dnp no)
@@
 			)
 		)
+		(property "LCSC" "C2869313"
+			(at 67.31 205.74 0)
+			(effects
+				(font
+					(size 1.27 1.27)
+				)
+				(hide yes)
+			)
+		)
 		(pin "1"
 		)
@@
 		(unit 1)
 		(exclude_from_sim no)
-		(in_bom no)
+		(in_bom yes)
 		(on_board yes)
 		(dnp no)
@@
 			)
 		)
+		(property "LCSC" "C552950"
+			(at 325.12 109.22 90)
+			(effects
+				(font
+					(size 1.27 1.27)
+				)
+				(hide yes)
+			)
+		)
 		(pin "1"
 		)
@@
 			)
 		)
-		(property "LCSC" "C22113"
+		(property "LCSC" "C189217"
 			(at 342.9 104.14 0)
 			(effects
@@
 		(unit 1)
 		(exclude_from_sim no)
-		(in_bom no)
+		(in_bom yes)
 		(on_board yes)
 		(dnp no)
@@
 			)
 		)
+		(property "LCSC" "C636381"
+			(at 71.12 242.57 0)
+			(effects
+				(font
+					(size 1.27 1.27)
+				)
+				(hide yes)
+			)
+		)
 		(pin "1"
 		)
@@
 			)
 		)
-		(property "LCSC" "C22113"
+		(property "LCSC" "C189217"
 			(at 328.93 149.86 0)
 			(effects
@@
 			)
 		)
-		(property "LCSC" "C2841056"
+		(property "LCSC" "C2871822"
 			(at 54.61 31.75 0)
 			(effects
